Commit message: Expand Gazebo Braccio simulation

File: ros2_ws/src/unoq_braccio_sim/urdf/braccio.urdf.xacro (robot description, xacro)
@@ -2,12 +2,35 @@
 <robot xmlns:xacro="http://www.ros.org/wiki/xacro" name="unoq_braccio">
   <xacro:property name="pi" value="3.14159265359"/>
+  <xacro:arg name="controllers_file" default=""/>
+  <material name="braccio_blue"><color rgba="0.05 0.18 0.8 1"/></material>
+  <material name="braccio_orange"><color rgba="0.94 0.6 0.05 1"/></material>
+  <material name="braccio_white"><color rgba="0.92 0.92 0.92 1"/></material>
+  <material name="braccio_dark"><color rgba="0.12 0.14 0.18 1"/></material>
+  <material name="camera_black"><color rgba="0.02 0.02 0.025 1"/></material>
+  <xacro:macro name="box_inertial" params="mass x y z">
+    <inertial>
+      <mass value="${mass}"/>
+      <inertia
+        ixx="${mass * (y * y + z * z) / 12.0}"
+        iyy="${mass * (x * x + z * z) / 12.0}"
+        izz="${mass * (x * x + y * y) / 12.0}"
+        ixy="0" ixz="0" iyz="0"/>
+    </inertial>
+  </xacro:macro>
   <link name="world"/>
   <link name="base_link">
     <visual>
-      <geometry><cylinder radius="0.06" length="0.04"/></geometry>
-      <material name="braccio_blue"><color rgba="0.05 0.18 0.8 1"/></material>
+      <origin xyz="0 0 0.02"/>
+      <geometry><cylinder radius="0.07" length="0.04"/></geometry>
+      <material name="braccio_blue"/>
     </visual>
-    <collision><geometry><cylinder radius="0.06" length="0.04"/></geometry></collision>
-    <inertial><mass value="0.4"/><inertia ixx="0.001" iyy="0.001" izz="0.001" ixy="0" ixz="0" iyz="0"/></inertial>
+    <collision>
+      <origin xyz="0 0 0.02"/>
+      <geometry><cylinder radius="0.07" length="0.04"/></geometry>
+    </collision>
+    <inertial>
+      <mass value="0.5"/>
+      <inertia ixx="0.0012" iyy="0.0012" izz="0.0012" ixy="0" ixz="0" iyz="0"/>
+    </inertial>
   </link>
   <joint name="base_fixed" type="fixed">
@@ -15,30 +38,62 @@
     <child link="base_link"/>
   </joint>
-  <xacro:macro name="arm_link" params="name length radius color">
+  <xacro:macro name="arm_box" params="name length width height material">
     <link name="${name}">
       <visual>
-        <origin xyz="${length / 2} 0 0" rpy="0 ${pi / 2} 0"/>
-        <geometry><cylinder radius="${radius}" length="${length}"/></geometry>
-        <material name="${name}_mat"><color rgba="${color}"/></material>
+        <origin xyz="${length / 2.0} 0 0"/>
+        <geometry><box size="${length} ${width} ${height}"/></geometry>
+        <material name="${material}"/>
       </visual>
       <collision>
-        <origin xyz="${length / 2} 0 0" rpy="0 ${pi / 2} 0"/>
-        <geometry><cylinder radius="${radius}" length="${length}"/></geometry>
+        <origin xyz="${length / 2.0} 0 0"/>
+        <geometry><box size="${length} ${width} ${height}"/></geometry>
       </collision>
-      <inertial>
-        <origin xyz="${length / 2} 0 0"/>
-        <mass value="0.15"/>
-        <inertia ixx="0.0004" iyy="0.0004" izz="0.0004" ixy="0" ixz="0" iyz="0"/>
-      </inertial>
+      <xacro:box_inertial mass="0.16" x="${length}" y="${width}" z="${height}"/>
     </link>
   </xacro:macro>
-  <xacro:arm_link name="shoulder_link" length="0.12" radius="0.018" color="0.94 0.6 0.05 1"/>
-  <xacro:arm_link name="elbow_link" length="0.12" radius="0.016" color="0.08 0.45 0.85 1"/>
-  <xacro:arm_link name="wrist_link" length="0.08" radius="0.014" color="0.92 0.92 0.92 1"/>
-  <xacro:arm_link name="gripper_link" length="0.05" radius="0.01" color="0.15 0.15 0.15 1"/>
+  <xacro:arm_box name="shoulder_link" length="0.125" width="0.036" height="0.036" material="braccio_orange"/>
+  <xacro:arm_box name="elbow_link" length="0.125" width="0.032" height="0.032" material="braccio_blue"/>
+  <xacro:arm_box name="wrist_link" length="0.075" width="0.028" height="0.028" material="braccio_white"/>
+  <xacro:arm_box name="wrist_rotate_link" length="0.035" width="0.03" height="0.03" material="braccio_dark"/>
+  <xacro:arm_box name="gripper_carriage" length="0.04" width="0.04" height="0.024" material="braccio_dark"/>
+  <link name="left_finger">
+    <visual>
+      <origin xyz="0.035 0.018 0"/>
+      <geometry><box size="0.07 0.012 0.014"/></geometry>
+      <material name="braccio_white"/>
+    </visual>
+    <collision>
+      <origin xyz="0.035 0.018 0"/>
+      <geometry><box size="0.07 0.012 0.014"/></geometry>
+    </collision>
+    <xacro:box_inertial mass="0.03" x="0.07" y="0.012" z="0.014"/>
+  </link>
+  <link name="right_finger">
+    <visual>
+      <origin xyz="0.035 -0.018 0"/>
+      <geometry><box size="0.07 0.012 0.014"/></geometry>
+      <material name="braccio_white"/>
+    </visual>
+    <collision>
+      <origin xyz="0.035 -0.018 0"/>
+      <geometry><box size="0.07 0.012 0.014"/></geometry>
+    </collision>
+    <xacro:box_inertial mass="0.03" x="0.07" y="0.012" z="0.014"/>
+  </link>
+  <link name="camera_link">
+    <visual>
+      <origin xyz="0 0 0"/>
+      <geometry><box size="0.03 0.022 0.018"/></geometry>
+      <material name="camera_black"/>
+    </visual>
+    <collision>
+      <geometry><box size="0.03 0.022 0.018"/></geometry>
+    </collision>
+    <xacro:box_inertial mass="0.04" x="0.03" y="0.022" z="0.018"/>
+  </link>
   <joint name="base" type="revolute">
     <parent link="base_link"/>
     <child link="shoulder_link"/>
-    <origin xyz="0 0 0.04"/>
+    <origin xyz="0 0 0.055"/>
     <axis xyz="0 0 1"/>
     <limit lower="-1.5708" upper="1.5708" effort="2" velocity="1"/>
@@ -47,5 +102,5 @@
     <parent link="shoulder_link"/>
     <child link="elbow_link"/>
-    <origin xyz="0.12 0 0"/>
+    <origin xyz="0.125 0 0"/>
     <axis xyz="0 1 0"/>
     <limit lower="-1.309" upper="1.309" effort="2" velocity="1"/>
@@ -54,5 +109,5 @@
     <parent link="elbow_link"/>
     <child link="wrist_link"/>
-    <origin xyz="0.12 0 0"/>
+    <origin xyz="0.125 0 0"/>
     <axis xyz="0 1 0"/>
     <limit lower="-1.5708" upper="1.5708" effort="2" velocity="1"/>
@@ -60,8 +115,72 @@
   <joint name="wrist_vertical" type="revolute">
     <parent link="wrist_link"/>
-    <child link="gripper_link"/>
-    <origin xyz="0.08 0 0"/>
+    <child link="wrist_rotate_link"/>
+    <origin xyz="0.075 0 0"/>
     <axis xyz="0 1 0"/>
     <limit lower="-1.5708" upper="1.5708" effort="1" velocity="1"/>
   </joint>
+  <joint name="wrist_rotation" type="revolute">
+    <parent link="wrist_rotate_link"/>
+    <child link="gripper_carriage"/>
+    <origin xyz="0.035 0 0"/>
+    <axis xyz="1 0 0"/>
+    <limit lower="-1.5708" upper="1.5708" effort="1" velocity="1"/>
+  </joint>
+  <joint name="gripper" type="prismatic">
+    <parent link="gripper_carriage"/>
+    <child link="left_finger"/>
+    <origin xyz="0.035 0 0"/>
+    <axis xyz="0 1 0"/>
+    <limit lower="0" upper="0.035" effort="1" velocity="0.05"/>
+  </joint>
+  <joint name="right_finger_fixed" type="fixed">
+    <parent link="gripper_carriage"/>
+    <child link="right_finger"/>
+    <origin xyz="0.035 0 0"/>
+  </joint>
+  <joint name="camera_mount" type="fixed">
+    <parent link="gripper_carriage"/>
+    <child link="camera_link"/>
+    <origin xyz="0.045 0 0.035" rpy="0 0 0"/>
+  </joint>
+  <ros2_control name="GazeboSystem" type="system">
+    <hardware>
+      <plugin>gazebo_ros2_control/GazeboSystem</plugin>
+    </hardware>
+    <joint name="base">
+      <command_interface name="position"/>
+      <state_interface name="position"/>
+      <state_interface name="velocity"/>
+    </joint>
+    <joint name="shoulder">
+      <command_interface name="position"/>
+      <state_interface name="position"/>
+      <state_interface name="velocity"/>
+    </joint>
+    <joint name="elbow">
+      <command_interface name="position"/>
+      <state_interface name="position"/>
+      <state_interface name="velocity"/>
+    </joint>
+    <joint name="wrist_vertical">
+      <command_interface name="position"/>
+      <state_interface name="position"/>
+      <state_interface name="velocity"/>
+    </joint>
+    <joint name="wrist_rotation">
+      <command_interface name="position"/>
+      <state_interface name="position"/>
+      <state_interface name="velocity"/>
+    </joint>
+    <joint name="gripper">
+      <command_interface name="position"/>
+      <state_interface name="position"/>
+      <state_interface name="velocity"/>
+    </joint>
+  </ros2_control>
+  <gazebo>
+    <plugin filename="libgazebo_ros2_control.so" name="gazebo_ros2_control">
+      <parameters>$(arg controllers_file)</parameters>
+    </plugin>
+  </gazebo>
 </robot>

Commit message: Remove duplicate xacro pi symbol

File: ros2_ws/src/unoq_braccio_sim/urdf/braccio.urdf.xacro (robot description, xacro)
@@ -1,5 +1,4 @@
 <?xml version="1.0"?>
 <robot xmlns:xacro="http://www.ros.org/wiki/xacro" name="unoq_braccio">
-  <xacro:property name="pi" value="3.14159265359"/>
   <xacro:arg name="controllers_file" default=""/>
   <material name="braccio_blue"><color rgba="0.05 0.18 0.8 1"/></material>

Commit message: Align Gazebo Braccio meshes with source model

File: ros2_ws/src/unoq_braccio_sim/urdf/braccio.urdf.xacro (robot description, xacro)
@@ -3,10 +3,7 @@
   <xacro:arg name="controllers_file" default=""/>
   <xacro:arg name="mesh_dir" default=""/>
-  <material name="braccio_orange"><color rgba="1.0 0.34 0.02 1"/></material>
-  <material name="braccio_orange_dark"><color rgba="0.76 0.18 0.02 1"/></material>
-  <material name="braccio_white"><color rgba="0.94 0.94 0.9 1"/></material>
-  <material name="braccio_metal"><color rgba="0.72 0.72 0.68 1"/></material>
-  <material name="braccio_black"><color rgba="0.03 0.035 0.045 1"/></material>
-  <material name="camera_black"><color rgba="0.01 0.01 0.015 1"/></material>
+  <material name="orange"><color rgba="1.0 0.34 0.02 1"/></material>
+  <material name="white"><color rgba="0.86 0.86 0.82 1"/></material>
+  <material name="black"><color rgba="0.02 0.02 0.025 1"/></material>
   <material name="lens_blue"><color rgba="0.08 0.28 0.55 1"/></material>
   <xacro:macro name="box_inertial" params="mass x y z">
@@ -20,18 +17,4 @@
     </inertial>
   </xacro:macro>
-  <xacro:macro name="joint_hub_visual" params="x y z radius material">
-    <visual>
-      <origin xyz="${x} ${y} ${z}" rpy="1.5708 0 0"/>
-      <geometry><cylinder radius="${radius}" length="0.018"/></geometry>
-      <material name="${material}"/>
-    </visual>
-  </xacro:macro>
-  <xacro:macro name="servo_box_visual" params="x y z sx sy sz">
-    <visual>
-      <origin xyz="${x} ${y} ${z}"/>
-      <geometry><box size="${sx} ${sy} ${sz}"/></geometry>
-      <material name="braccio_black"/>
-    </visual>
-  </xacro:macro>
   <xacro:macro name="mesh_visual" params="filename material x y z rr rp ry">
     <visual>
@@ -43,24 +26,16 @@
     </visual>
   </xacro:macro>
-  <xacro:macro name="paired_arm_link" params="name length plate_height plate_thickness y_offset mesh mesh_x mesh_y mesh_z">
-    <link name="${name}">
-      <xacro:mesh_visual filename="${mesh}" material="braccio_orange" x="${mesh_x}" y="${mesh_y}" z="${mesh_z}" rr="0" rp="0" ry="0"/>
-      <collision>
-        <origin xyz="${length / 2.0} 0 0"/>
-        <geometry><box size="${length} ${y_offset * 2.0 + plate_thickness} ${plate_height}"/></geometry>
-      </collision>
-      <xacro:box_inertial mass="0.18" x="${length}" y="${y_offset * 2.0 + plate_thickness}" z="${plate_height}"/>
-    </link>
-  </xacro:macro>
   <link name="world"/>
   <link name="base_link">
-    <xacro:mesh_visual filename="braccio_base.stl" material="braccio_orange" x="0" y="0.004" z="0.04" rr="0" rp="0" ry="3.1416"/>
-    <collision>
-      <origin xyz="0 0 0.045"/>
-      <geometry><cylinder radius="0.09" length="0.09"/></geometry>
+    <visual>
+      <geometry><cylinder length="0.01" radius="0.053"/></geometry>
+      <material name="black"/>
+    </visual>
+    <collision>
+      <geometry><cylinder length="0.01" radius="0.053"/></geometry>
     </collision>
     <inertial>
-      <mass value="0.7"/>
-      <inertia ixx="0.002" iyy="0.002" izz="0.002" ixy="0" ixz="0" iyz="0"/>
+      <mass value="2"/>
+      <inertia ixx="0.015" ixy="0" ixz="0" iyy="0.00666666666667" iyz="0" izz="0.0216666666667"/>
     </inertial>
   </link>
@@ -69,44 +44,59 @@
     <child link="base_link"/>
   </joint>
-  <xacro:paired_arm_link name="shoulder_link" length="0.14" plate_height="0.035" plate_thickness="0.012" y_offset="0.035" mesh="braccio_shoulder.stl" mesh_x="-0.0045" mesh_y="0.0055" mesh_z="-0.026"/>
-  <xacro:paired_arm_link name="elbow_link" length="0.13" plate_height="0.03" plate_thickness="0.01" y_offset="0.03" mesh="braccio_elbow.stl" mesh_x="-0.0045" mesh_y="0.005" mesh_z="-0.025"/>
-  <xacro:paired_arm_link name="wrist_link" length="0.075" plate_height="0.026" plate_thickness="0.01" y_offset="0.024" mesh="braccio_wrist_pitch.stl" mesh_x="0.003" mesh_y="-0.0004" mesh_z="-0.024"/>
-  <link name="wrist_rotate_link">
-    <xacro:mesh_visual filename="braccio_wrist_roll.stl" material="braccio_white" x="0.006" y="0" z="0" rr="0" rp="0" ry="0"/>
-    <collision>
-      <origin xyz="0.028 0 0"/>
-      <geometry><box size="0.05 0.05 0.035"/></geometry>
-    </collision>
-    <xacro:box_inertial mass="0.12" x="0.05" y="0.05" z="0.035"/>
-  </link>
-  <link name="gripper_carriage">
-    <visual>
-      <origin xyz="0.02 0 0"/>
-      <geometry><box size="0.04 0.05 0.025"/></geometry>
-      <material name="braccio_white"/>
-    </visual>
-    <visual>
-      <origin xyz="0.01 0 0.022"/>
-      <geometry><cylinder radius="0.019" length="0.018"/></geometry>
-      <material name="braccio_metal"/>
-    </visual>
-    <collision>
-      <origin xyz="0.02 0 0"/>
-      <geometry><box size="0.04 0.05 0.025"/></geometry>
-    </collision>
-    <xacro:box_inertial mass="0.1" x="0.04" y="0.05" z="0.025"/>
-  </link>
-  <link name="left_finger">
-    <xacro:mesh_visual filename="braccio_left_gripper.stl" material="braccio_white" x="0" y="-0.012" z="0" rr="0" rp="1.5708" ry="0"/>
-    <collision>
-      <origin xyz="0.04 0.024 0"/>
+  <link name="braccio_base_link">
+    <xacro:mesh_visual filename="braccio_base.stl" material="orange" x="0" y="0.004" z="0" rr="0" rp="0" ry="3.1416"/>
+    <collision>
+      <origin xyz="0 0 0.035"/>
+      <geometry><cylinder radius="0.065" length="0.07"/></geometry>
+    </collision>
+    <inertial>
+      <mass value="2"/>
+      <inertia ixx="0.015" ixy="0" ixz="0" iyy="0.00666666666667" iyz="0" izz="0.0216666666667"/>
+    </inertial>
+  </link>
+  <link name="shoulder_link">
+    <xacro:mesh_visual filename="braccio_shoulder.stl" material="orange" x="-0.0045" y="0.0055" z="-0.026" rr="0" rp="0" ry="0"/>
+    <collision>
+      <origin xyz="0 0 0.06"/>
+      <geometry><box size="0.055 0.08 0.12"/></geometry>
+    </collision>
+    <xacro:box_inertial mass="0.1" x="0.055" y="0.08" z="0.12"/>
+  </link>
+  <link name="elbow_link">
+    <xacro:mesh_visual filename="braccio_elbow.stl" material="orange" x="-0.0045" y="0.005" z="-0.025" rr="0" rp="0" ry="0"/>
+    <collision>
+      <origin xyz="0 0 0.06"/>
+      <geometry><box size="0.05 0.07 0.12"/></geometry>
+    </collision>
+    <xacro:box_inertial mass="0.1" x="0.05" y="0.07" z="0.12"/>
+  </link>
+  <link name="wrist_pitch_link">
+    <xacro:mesh_visual filename="braccio_wrist_pitch.stl" material="orange" x="0.003" y="-0.0004" z="-0.024" rr="0" rp="0" ry="0"/>
+    <collision>
+      <origin xyz="0 0 0.035"/>
+      <geometry><box size="0.045 0.055 0.07"/></geometry>
+    </collision>
+    <xacro:box_inertial mass="0.08" x="0.045" y="0.055" z="0.07"/>
+  </link>
+  <link name="wrist_roll_link">
+    <xacro:mesh_visual filename="braccio_wrist_roll.stl" material="white" x="0.006" y="0" z="0" rr="0" rp="0" ry="0"/>
+    <collision>
+      <origin xyz="0 0 0.018"/>
+      <geometry><box size="0.045 0.045 0.04"/></geometry>
+    </collision>
+    <xacro:box_inertial mass="0.08" x="0.045" y="0.045" z="0.04"/>
+  </link>
+  <link name="right_gripper_link">
+    <xacro:mesh_visual filename="braccio_right_gripper.stl" material="white" x="0" y="-0.012" z="0.010" rr="0" rp="1.5708" ry="0"/>
+    <collision>
+      <origin xyz="0.035 -0.012 0.01"/>
       <geometry><box size="0.08 0.012 0.014"/></geometry>
     </collision>
     <xacro:box_inertial mass="0.03" x="0.08" y="0.012" z="0.014"/>
   </link>
-  <link name="right_finger">
-    <xacro:mesh_visual filename="braccio_right_gripper.stl" material="braccio_white" x="0" y="-0.012" z="0.010" rr="0" rp="1.5708" ry="0"/>
-    <collision>
-      <origin xyz="0.04 -0.024 0"/>
+  <link name="left_gripper_link">
+    <xacro:mesh_visual filename="braccio_left_gripper.stl" material="white" x="0" y="-0.012" z="0" rr="0" rp="1.5708" ry="0"/>
+    <collision>
+      <origin xyz="0.035 -0.012 0"/>
       <geometry><box size="0.08 0.012 0.014"/></geometry>
     </collision>
@@ -117,5 +107,5 @@
       <origin xyz="0 0 0"/>
       <geometry><box size="0.034 0.026 0.022"/></geometry>
-      <material name="camera_black"/>
+      <material name="black"/>
     </visual>
     <visual>
@@ -124,60 +114,68 @@
       <material name="lens_blue"/>
     </visual>
-    <collision>
-      <geometry><box size="0.034 0.026 0.022"/></geometry>
-    </collision>
+    <collision><geometry><box size="0.034 0.026 0.022"/></geometry></collision>
     <xacro:box_inertial mass="0.04" x="0.034" y="0.026" z="0.022"/>
   </link>
   <joint name="base" type="revolute">
+    <axis xyz="0 0 1"/>
+    <limit effort="2" lower="-1.5708" upper="1.5708" velocity="1"/>
+    <origin xyz="0 0 0" rpy="0 0 0"/>
     <parent link="base_link"/>
+    <child link="braccio_base_link"/>
+    <dynamics damping="0.1" friction="0.001"/>
+  </joint>
+  <joint name="shoulder" type="revolute">
+    <axis xyz="1 0 0"/>
+    <limit effort="2" lower="-1.309" upper="1.309" velocity="1"/>
+    <origin xyz="0 -0.002 0.072" rpy="-1.5708 0 0"/>
+    <parent link="braccio_base_link"/>
     <child link="shoulder_link"/>
-    <origin xyz="0 0 0.11"/>
-    <axis xyz="0 0 1"/>
-    <limit lower="-1.5708" upper="1.5708" effort="2" velocity="1"/>
-  </joint>
-  <joint name="shoulder" type="revolute">
+    <dynamics damping="0.1" friction="0.001"/>
+  </joint>
+  <joint name="elbow" type="revolute">
+    <axis xyz="1 0 0"/>
+    <limit effort="2" lower="-1.5708" upper="1.5708" velocity="1"/>
+    <origin xyz="0 0 0.125" rpy="-1.5708 0 0"/>
     <parent link="shoulder_link"/>
     <child link="elbow_link"/>
-    <origin xyz="0.14 0 0"/>
+    <dynamics damping="0.1" friction="0.001"/>
+  </joint>
+  <joint name="wrist_vertical" type="revolute">
+    <axis xyz="1 0 0"/>
+    <limit effort="1" lower="-1.5708" upper="1.5708" velocity="1"/>
+    <origin xyz="0 0 0.125" rpy="-1.5708 0 0"/>
+    <parent link="elbow_link"/>
+    <child link="wrist_pitch_link"/>
+    <dynamics damping="0.1" friction="0.001"/>
+  </joint>
+  <joint name="wrist_rotation" type="revolute">
+    <axis xyz="0 0 -1"/>
+    <limit effort="1" lower="-1.5708" upper="1.5708" velocity="1"/>
+    <origin xyz="0 0 0.06" rpy="0 0 1.5708"/>
+    <parent link="wrist_pitch_link"/>
+    <child link="wrist_roll_link"/>
+    <dynamics damping="0.1" friction="0.001"/>
+  </joint>
+  <joint name="gripper" type="revolute">
+    <axis xyz="0 -1 0"/>
+    <limit effort="1" lower="0.1750" upper="1.2741" velocity="1"/>
+    <origin xyz="0.010 0 0.03" rpy="0 -0.2967 0"/>
+    <parent link="wrist_roll_link"/>
+    <child link="right_gripper_link"/>
+    <dynamics damping="0.1" friction="0.001"/>
+  </joint>
+  <joint name="left_gripper_mimic" type="revolute">
     <axis xyz="0 1 0"/>
-    <limit lower="-1.309" upper="1.309" effort="2" velocity="1"/>
-  </joint>
-  <joint name="elbow" type="revolute">
-    <parent link="elbow_link"/>
-    <child link="wrist_link"/>
-    <origin xyz="0.13 0 0"/>
-    <axis xyz="0 1 0"/>
-    <limit lower="-1.5708" upper="1.5708" effort="2" velocity="1"/>
-  </joint>
-  <joint name="wrist_vertical" type="revolute">
-    <parent link="wrist_link"/>
-    <child link="wrist_rotate_link"/>
-    <origin xyz="0.075 0 0"/>
-    <axis xyz="0 1 0"/>
-    <limit lower="-1.5708" upper="1.5708" effort="1" velocity="1"/>
-  </joint>
-  <joint name="wrist_rotation" type="revolute">
-    <parent link="wrist_rotate_link"/>
-    <child link="gripper_carriage"/>
-    <origin xyz="0.045 0 0"/>
-    <axis xyz="1 0 0"/>
-    <limit lower="-1.5708" upper="1.5708" effort="1" velocity="1"/>
-  </joint>
-  <joint name="gripper" type="prismatic">
-    <parent link="gripper_carriage"/>
-    <child link="left_finger"/>
-    <origin xyz="0.04 0 0"/>
-    <axis xyz="0 1 0"/>
-    <limit lower="0" upper="0.035" effort="1" velocity="0.05"/>
-  </joint>
-  <joint name="right_finger_fixed" type="fixed">
-    <parent link="gripper_carriage"/>
-    <child link="right_finger"/>
-    <origin xyz="0.04 0 0"/>
+    <mimic joint="gripper"/>
+    <limit effort="1" lower="1.2741" upper="2.3732" velocity="1"/>
+    <origin xyz="-0.010 0 0.03" rpy="0 3.4383 0"/>
+    <parent link="wrist_roll_link"/>
+    <child link="left_gripper_link"/>
+    <dynamics damping="0.1" friction="0.001"/>
   </joint>
   <joint name="camera_mount" type="fixed">
-    <parent link="gripper_carriage"/>
+    <parent link="wrist_roll_link"/>
     <child link="camera_link"/>
-    <origin xyz="0.052 0 0.04" rpy="0 0 0"/>
+    <origin xyz="0.03 0 0.055" rpy="0 0 0"/>
   </joint>
   <ros2_control name="GazeboSystem" type="system">

Commit message: Anchor Braccio sim spawn at world origin

File: ros2_ws/src/unoq_braccio_sim/urdf/braccio.urdf.xacro (robot description, xacro)
@@ -43,4 +43,5 @@
     <parent link="world"/>
     <child link="base_link"/>
+    <origin xyz="0 0 0.02" rpy="0 0 0"/>
   </joint>
   <link name="braccio_base_link">
@@ -120,5 +121,5 @@
     <axis xyz="0 0 1"/>
     <limit effort="2" lower="-1.5708" upper="1.5708" velocity="1"/>
-    <origin xyz="0 0 0" rpy="0 0 0"/>
+    <origin xyz="0 0 0.01" rpy="0 0 0"/>
     <parent link="base_link"/>
     <child link="braccio_base_link"/>

Commit message: Fix Gazebo Braccio base inertias

File: ros2_ws/src/unoq_braccio_sim/urdf/braccio.urdf.xacro (robot description, xacro)
@@ -37,5 +37,5 @@
     <inertial>
       <mass value="2"/>
-      <inertia ixx="0.015" ixy="0" ixz="0" iyy="0.00666666666667" iyz="0" izz="0.0216666666667"/>
+      <inertia ixx="0.004" ixy="0" ixz="0" iyy="0.004" iyz="0" izz="0.004"/>
     </inertial>
   </link>
@@ -53,5 +53,5 @@
     <inertial>
       <mass value="2"/>
-      <inertia ixx="0.015" ixy="0" ixz="0" iyy="0.00666666666667" iyz="0" izz="0.0216666666667"/>
+      <inertia ixx="0.004" ixy="0" ixz="0" iyy="0.004" iyz="0" izz="0.004"/>
     </inertial>
   </link>
